Commit message: feat(description): finish robot core and inertial macros xacros files

File: my_bot_dev_ws/src/my_bot/description/robot_core.xacro (robot description, xacro)
@@ -1,6 +1,10 @@
 <?xml version="1.0"?>
 <robot xmlns:xacro="http://www.ros.org/wiki/xacro" >
+    <xacro:include filename="inertial_macros.xacro"/>
     <material name="white">
         <color rgba="1 1 1 1"/>
+    </material>
+    <material name="black">
+        <color rgba="0.0 0.0 0.0 1.0"/>
     </material>
     <material name="orange">
@@ -13,5 +17,98 @@
         <color rgba="0.1 0.1 0.1 1"/>
     </material>
+    <!-- BASE LINK-->
     <link name="base_link">
     </link>
+    <!-- CHASSIS LINK-->
+    <joint name="chassis_joint" type="fixed">
+        <parent link="base_link"/>
+        <child link="chassis"/>
+        <origin xyz="-0.1 0.0 0.0"/>
+    </joint>
+    <link name="chassis">
+        <visual>
+            <origin xyz="0.15 0.0 0.075"/>
+            <geometry>
+                <box size="0.3 0.3 0.15"/>
+            </geometry>
+            <material name="white"/>
+        </visual>
+        <collision>
+            <origin xyz="0.15 0.0 0.075"/>
+            <geometry>
+                <box size="0.3 0.3 0.15"/>
+            </geometry>
+        </collision>
+        <xacro:inertial_box mass="0.5" x="0.3" y="0.3" z="0.15">
+            <origin xyz="0.15 0.0 0.075" rpy="0.0 0.0 0.0"/>
+        </xacro:inertial_box>
+    </link>
+    <!-- LEFT WHEEL LINK-->
+    <joint name="left_wheel_joint" type="continuous">
+        <parent link="base_link"/>
+        <child link="left_wheel"/>
+        <origin xyz="0.0 0.175 0.0" rpy="-${pi / 2} 0.0 0.0"/>
+        <axis xyz="0.0 0.0 1"/>
+    </joint>
+    <link name="left_wheel">
+        <visual>
+            <geometry>
+                <cylinder radius="0.05" length="0.04"/>
+            </geometry>
+            <material name="blue"/>
+        </visual>
+        <collision>
+            <geometry>
+                <cylinder radius="0.05" length="0.04"/>
+            </geometry>
+        </collision>
+        <xacro:inertial_cylinder mass="0.1" length="0.04" radius="0.05">
+            <origin xyz="0.0 0.0 0.0" rpy="0.0 0.0 0.0"/>
+        </xacro:inertial_cylinder>
+    </link>
+    <!-- RIGHT WHEEL LINK-->
+    <joint name="right_wheel_joint" type="continuous">
+        <parent link="base_link"/>
+        <child link="right_wheel"/>
+        <origin xyz="0.0 -0.175 0.0" rpy="${pi / 2} 0.0 0.0"/>
+        <axis xyz="0.0 0.0 -1"/>
+    </joint>
+    <link name="right_wheel">
+        <visual>
+            <geometry>
+                <cylinder radius="0.05" length="0.04"/>
+            </geometry>
+            <material name="blue"/>
+        </visual>
+        <collision>
+            <geometry>
+                <cylinder radius="0.05" length="0.04"/>
+            </geometry>
+        </collision>
+        <xacro:inertial_cylinder mass="0.1" length="0.04" radius="0.05">
+            <origin xyz="0.0 0.0 0.0" rpy="0.0 0.0 0.0"/>
+        </xacro:inertial_cylinder>
+    </link>
+    <!-- CUSTER WHEEL LINK-->
+     <joint name="custer_wheel_joint" type="fixed">
+        <parent link="chassis"/>
+        <child link="custer_wheel"/>
+        <origin xyz="0.24 0.0 0.0"/>
+     </joint>
+     <link name="custer_wheel">
+        <visual>
+            <geometry>
+                <sphere radius="0.05"/>
+            </geometry>
+            <material name="black"/>
+        </visual>
+        <collision>
+            <geometry>
+                <sphere radius="0.05"/>
+            </geometry>
+        </collision>
+        <xacro:inertial_sphere mass="0.1" radius="0.05">
+            <origin xyz="0.0 0.0 0.0" rpy="0.0 0.0 0.0"/>
+        </xacro:inertial_sphere>
+     </link>
 </robot>

Commit message: feat(description): add gazebo references into robot_core.xacro

File: my_bot_dev_ws/src/my_bot/description/robot_core.xacro (robot description, xacro)
@@ -44,4 +44,7 @@
         </xacro:inertial_box>
     </link>
+        <!-- <gazebo reference="chassis">
+            <material>Gazebo/White</material>
+        </gazebo> -->
     <!-- LEFT WHEEL LINK-->
     <joint name="left_wheel_joint" type="continuous">
@@ -67,4 +70,7 @@
         </xacro:inertial_cylinder>
     </link>
+    <!-- <gazebo reference="left_wheel">
+        <material>Gazebo/Blue</material>
+    </gazebo> -->
     <!-- RIGHT WHEEL LINK-->
     <joint name="right_wheel_joint" type="continuous">
@@ -90,4 +96,7 @@
         </xacro:inertial_cylinder>
     </link>
+    <!-- <gazebo reference="right_wheel">
+        <material>Gazebo/Blue</material>
+    </gazebo> -->
     <!-- CUSTER WHEEL LINK-->
      <joint name="custer_wheel_joint" type="fixed">
@@ -112,3 +121,6 @@
         </xacro:inertial_sphere>
      </link>
+        <!-- <gazebo reference="custer_wheel">
+            <material>Gazebo/Black</material>
+        </gazebo> -->
 </robot>
